File: pcb/presence-sensor/presence-sensor.kicad_sch (KiCad schematic)
At the start: 35 parts, among them J1 Conn_Coaxial, J2 Conn_01x03_MountingPin, J3 USB_C_Receptacle_USB2.0_16P, SW1 SW_Push, SW2 SW_Push, U1 CC2340R52E0RGER, U2 SEN0609, U3 XC6206P332MR-G, Y1 48M, Y2 32k768

Commit message: rework VDDR and ERASE button
Parts:
- added C5, C6: 0u1, Capacitor_SMD:C_0603_1608Metric, symbol Device:C
- J2: value Conn_01x03_MountingPin -> RPI_DEBUG_PROBE
Connections:
- net +VDDR: now also C5.1, C6.1; no longer U1.17 (DCDC)
- net GND: now also C7.2, C5.2, C6.2; no longer C7.1
- net +VDDD: now reaches U1.16 (VDDD)
- net +VDDD: now also C7.1; no longer C7.2
- net SWDIO: now reaches J2.1 (Pin_1), U1.7 (DIO16_SWDIO)
- net SWCLK: now reaches J2.2 (Pin_2), U1.8 (DIO17_SWDCK)
- no-connect marks 10 -> 11
Other:
- note added: "Impedance matching taken from MCU datasheet"
- note added: "Jumpers are in case TX/RX is connected wrong"
- note added: "optionally replace with capacitor"
- moved on the sheet: C1, C10, C11, C12, C13, C14, C15, C17, C2, C3, C4, C7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

Commit message: part details
Parts:
- C1, C2, C3, C5, C6: DigiKey Part # (none) -> 311-1344-2-ND; MPN (none) -> CC0603KRX7R9BB104; Manufacturer (none) -> YAGEO; Mouser Part # (none) -> 603-CC603KRX7R9BB104
- C10, C4: DigiKey Part # (none) -> 1276-1192-2-ND; MPN (none) -> CL10A106KP8NNNC; Manufacturer (none) -> Samsung Electro-Mechanics; Mouser Part # (none) -> 187-CL10A106KP8NNNC
- C11, C12: DigiKey Part # (none) -> 1276-1296-2-ND; MPN (none) -> CL10C150JB8NNNC; Manufacturer (none) -> Samsung Electro-Mechanics; Mouser Part # (none) -> 187-CL10C150JB8NNNC
- C13, C17, C7, C8, C9: DigiKey Part # (none) -> 1276-1860-2-ND; MPN (none) -> CL10A105KB8NNNC; Manufacturer (none) -> Samsung Electro-Mechanics; Mouser Part # (none) -> 187-CL10A105KB8NNNC
- C14, C15: MPN (none) -> 0603CG1R5C500NT; Manufacturer (none) -> FH (Guangdong Fenghua Advanced Tech)
- J2: DigiKey Part # (none) -> 455-SM03B-SRSS-TBTR-ND; MPN (none) -> SM03B-SRSS-TB(LF)(SN); Manufacturer (none) -> JST; Mouser Part # (none) -> 306-SM03BSRSSTBLFSNP
- J3: DigiKey Part # (none) -> 2073-USB4105-GF-A-120TR-ND; MPN (none) -> USB4105-GF-A-120; Manufacturer (none) -> Global Connector Technology; Mouser Part # (none) -> 640-USB4105-GF-A-120
- L2: DigiKey Part # (none) -> 3442-SDCL1005C2N7STDFTR-ND; MPN (none) -> SDCL1005C2N7STDF; Manufacturer (none) -> Sunlord
- R1, R2, R3, R4, R5: MPN (none) -> 0603WAF1003T5E; Manufacturer (none) -> UNI-ROYAL(Uniroyal Elec); Mouser Part # (none) -> 303-0603WAF1003T5E
- R6: MPN (none) -> 0603WAF0000T5E; Manufacturer (none) -> UNI-ROYAL(Uniroyal Elec); Mouser Part # (none) -> 303-0603WAF0000T5E
- SW1, SW2: DigiKey Part # (none) -> SW1451TR-ND; MPN (none) -> B3U-1100PM; Manufacturer (none) -> Omron Electronics; Mouser Part # (none) -> 653-B3U-1100PM
- U1: DigiKey Part # (none) -> 296-CC2340R52E0RGERTR-ND; MPN (none) -> CC2340R52E0RGER; Manufacturer (none) -> Texas Instruments; Mouser Part # (none) -> 595-CC2340R52E0RGER
- U3: DigiKey Part # (none) -> 893-XC6206P332MR-GTR-ND; MPN (none) -> XC6206P332MR-G; Manufacturer (none) -> Torex Semicon; Mouser Part # (none) -> 865-XC6206P332MR-G
- Y1: DigiKey Part # (none) -> 4309-XC32M4-48.000-F08NLDTKTR-ND; MPN (none) -> XC32M4-48.000-F08NLDT; Manufacturer (none) -> HCI
- Y2: MPN (none) -> Q13FC13500049; Manufacturer (none) -> Seiko Epson; Mouser Part # (none) -> 732-532.7680KA-E
