File: pcb/presence-sensor.kicad_pcb (KiCad board)
At the start: 4 copper layers, 30 x 36 mm, 37 parts, among them J1 Conn_Coaxial, J2 RPI_DEBUG_PROBE, J3 USB_C_Receptacle_USB2.0_16P, SW1 SW_Push, SW2 SW_Push, U1 CC2340R52E0RGER, U2 SEN0609, U3 XC6206P332MR-G, Y1 48M, Y2 32k768

Commit message: finalize files
Parts:
- C1, C10, C11, C12, C13, C14, C15, C17, C2, C3, C4, C5, C6, C7, C8, C9: footprint Capacitor_SMD:C_0603_1608Metric -> footprints:C_0603_1608Metric
- H1, H2: footprint MountingHole:MountingHole_2.5mm -> footprints:MountingHole_2.5mm
- J1: footprint RF_Antenna:Texas_SWRA117D_2.4GHz_Right -> footprints:Texas_SWRA117D_2.4GHz_Right
- J2: footprint Connector_JST:JST_SH_SM03B-SRSS-TB_1x03-1MP_P1.00mm_Horizontal -> footprints:JST_SH_SM03B-SRSS-TB_1x03-1MP_P1.00mm_Horizontal
- J3: footprint Connector_USB:USB_C_Receptacle_GCT_USB4105-xx-A_16P_TopMnt_Horizontal -> footprints:USB_C_Receptacle_GCT_USB4105-xx-A_16P_TopMnt_Horizontal
- JP1, JP2: footprint Jumper:SolderJumper-2_P1.3mm_Bridged_RoundedPad1.0x1.5mm -> footprints:SolderJumper-2_P1.3mm_Bridged_RoundedPad1.0x1.5mm
- L2: footprint Inductor_SMD:L_0402_1005Metric -> footprints:L_0402_1005Metric
- R1, R2, R3, R4, R5, R6: footprint Resistor_SMD:R_0603_1608Metric -> footprints:R_0603_1608Metric
- SW1, SW2: footprint Button_Switch_SMD:SW_SPST_B3U-1100P -> footprints:SW_SPST_B3U-1100P
- U2: footprint Connector_PinHeader_2.54mm:PinHeader_1x05_P2.54mm_Vertical -> footprints:PinHeader_1x05_P2.54mm_Vertical
- U3: footprint Package_TO_SOT_SMD:SOT-23-3 -> footprints:SOT-23-3
- Y1: footprint Crystal:Crystal_SMD_3225-4Pin_3.2x2.5mm -> footprints:Crystal_SMD_3225-4Pin_3.2x2.5mm
- Y2: footprint Crystal:Crystal_SMD_3215-2Pin_3.2x1.5mm -> footprints:Crystal_SMD_3215-2Pin_3.2x1.5mm
