File: pcb/presence-sensor.kicad_sch (KiCad schematic)
At the start: 37 parts, among them J1 Conn_Coaxial, J2 RPI_DEBUG_PROBE, J3 USB_C_Receptacle_USB2.0_16P, SW1 SW_Push, SW2 SW_Push, U1 CC2340R52E0RGER, U2 SEN0609, U3 XC6206P332MR-G, Y1 48M, Y2 32k768

Commit message: finalize files
Parts:
- C1, C10, C11, C12, C13, C14, C15, C17, C2, C3, C4, C5, C6, C7, C8, C9: footprint Capacitor_SMD:C_0603_1608Metric -> footprints:C_0603_1608Metric; symbol Device:C -> presence-sensor:C
- H1, H2: footprint MountingHole:MountingHole_2.5mm -> footprints:MountingHole_2.5mm; symbol Mechanical:MountingHole -> presence-sensor:MountingHole
- J1: footprint RF_Antenna:Texas_SWRA117D_2.4GHz_Right -> footprints:Texas_SWRA117D_2.4GHz_Right; symbol Connector:Conn_Coaxial -> presence-sensor:Conn_Coaxial
- J2: footprint Connector_JST:JST_SH_SM03B-SRSS-TB_1x03-1MP_P1.00mm_Horizontal -> footprints:JST_SH_SM03B-SRSS-TB_1x03-1MP_P1.00mm_Horizontal; symbol Connector_Generic_MountingPin:Conn_01x03_MountingPin -> presence-sensor:Conn_01x03_MountingPin
- J3: footprint Connector_USB:USB_C_Receptacle_GCT_USB4105-xx-A_16P_TopMnt_Horizontal -> footprints:USB_C_Receptacle_GCT_USB4105-xx-A_16P_TopMnt_Horizontal; symbol Connector:USB_C_Receptacle_USB2.0_16P -> presence-sensor:USB_C_Receptacle_USB2.0_16P
- JP1, JP2: footprint Jumper:SolderJumper-2_P1.3mm_Bridged_RoundedPad1.0x1.5mm -> footprints:SolderJumper-2_P1.3mm_Bridged_RoundedPad1.0x1.5mm; symbol Jumper:SolderJumper_2_Bridged -> presence-sensor:SolderJumper_2_Bridged
- L2: footprint Inductor_SMD:L_0402_1005Metric -> footprints:L_0402_1005Metric; symbol Device:L -> presence-sensor:L
- R1, R2, R3, R4, R5, R6: footprint Resistor_SMD:R_0603_1608Metric -> footprints:R_0603_1608Metric; symbol Device:R -> presence-sensor:R
- SW1, SW2: footprint Button_Switch_SMD:SW_SPST_B3U-1100P -> footprints:SW_SPST_B3U-1100P; symbol Switch:SW_Push -> presence-sensor:SW_Push
- U2: footprint Connector_PinHeader_2.54mm:PinHeader_1x05_P2.54mm_Vertical -> footprints:PinHeader_1x05_P2.54mm_Vertical
- U3: footprint Package_TO_SOT_SMD:SOT-23-3 -> footprints:SOT-23-3; symbol Regulator_Linear:XC6206PxxxMR -> presence-sensor:XC6206PxxxMR
- Y1: footprint Crystal:Crystal_SMD_3225-4Pin_3.2x2.5mm -> footprints:Crystal_SMD_3225-4Pin_3.2x2.5mm; symbol Device:Crystal_GND24 -> presence-sensor:Crystal_GND24
- Y2: footprint Crystal:Crystal_SMD_3215-2Pin_3.2x1.5mm -> footprints:Crystal_SMD_3215-2Pin_3.2x1.5mm; symbol Device:Crystal -> presence-sensor:Crystal
